File: pcb/_autosave-EngineManagement.kicad_pcb (KiCad board)
At the start: 2 copper layers, 97 x 56.1 mm, 47 parts, among them K1 Temps, K5 FuelCool, K6 FuelCoolAlt, K7 Supply, U1 LM7808CT, U3 ArdinoMinPro, U5 MCP2515Shield

Commit message: Redesigned to not use VP J1939 instruments
Parts:
- moved REF** 8.13 mm to (100.8, 94.2)
- moved REF** 8.13 mm to (100.8, 48.8)
- moved REF** 5.61 mm to (191.3, 94.2)
- moved REF** 5.59 mm to (191.5, 48.5)
Changed lines of the file:
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@@
     (links 83)
     (no_connects 0)
-    (area 96.952999 42.850999 194.131001 99.135001)
+    (area 39.017498 13.807691 195.426001 272.896001)
     (thickness 1.6)
-    (drawings 20)
+    (drawings 21)
     (tracks 277)
     (zones 0)
@@
     (pad_drill 0.762)
     (pad_to_mask_clearance 0.2)
-    (aux_axis_origin 104.394 142.494)
+    (aux_axis_origin 96.774 99.568)
     (grid_origin 97.79 42.164)
     (visible_elements FFFFFF7F)
@@
   )
   (module Connect:1pin (layer F.Cu)
-    (at 185.928 48.514)
+    (at 191.516 48.514)
     (descr "module 1 pin (ou trou mecanique de percage)")
     (tags DEV)
@@
   )
   (module Connect:1pin (layer F.Cu)
-    (at 185.674 93.726)
+    (at 191.262 94.234)
     (descr "module 1 pin (ou trou mecanique de percage)")
     (tags DEV)
@@
   )
   (module Connect:1pin (layer F.Cu)
-    (at 108.966 94.234)
+    (at 100.838 94.234)
     (descr "module 1 pin (ou trou mecanique de percage)")
     (tags DEV)
@@
   )
   (module Connect:1pin (layer F.Cu)
-    (at 108.966 48.768)
+    (at 100.838 48.768)
     (descr "module 1 pin (ou trou mecanique de percage)")
     (tags DEV)
@@
     (fp_circle (center 0 0) (end 0 -2.286) (layer F.SilkS) (width 0.15))
     (pad 1 thru_hole circle (at 0 0) (size 4.064 4.064) (drill 3.048) (layers *.Cu *.Mask))
+  )
+  (dimension 77.216 (width 0.3) (layer Dwgs.User)
+    (gr_text "77.216 mm" (at 147.574 29.384) (layer Dwgs.User)
+      (effects (font (size 1.5 1.5) (thickness 0.3)))
+    )
+    (feature1 (pts (xy 186.182 42.926) (xy 186.182 28.034)))
+    (feature2 (pts (xy 108.966 42.926) (xy 108.966 28.034)))
+    (crossbar (pts (xy 108.966 30.734) (xy 186.182 30.734)))
+    (arrow1a (pts (xy 186.182 30.734) (xy 185.055496 31.320421)))
+    (arrow1b (pts (xy 186.182 30.734) (xy 185.055496 30.147579)))
+    (arrow2a (pts (xy 108.966 30.734) (xy 110.092504 31.320421)))
+    (arrow2b (pts (xy 108.966 30.734) (xy 110.092504 30.147579)))
   )
   (gr_line (start 195.326 94.234) (end 195.326 92.202) (angle 90) (layer Dwgs.User) (width 0.2))
@@
   (segment (start 116.335 59.439) (end 119.888 59.439) (width 1) (layer F.Cu) (net 1))
   (segment (start 129.032 59.69) (end 110.998 59.69) (width 1) (layer B.Cu) (net 2))
-  (segment (start 110.998 59.69) (end 108.966 57.658) (width 1) (layer B.Cu) (net 2) (status 800000))
+  (segment (start 110.998 59.69) (end 108.966 57.658) (width 1) (layer B.Cu) (net 2))
   (segment (start 147.574 56.134) (end 152.908 56.134) (width 1) (layer B.Cu) (net 2))
   (segment (start 177.419 81.661) (end 180.133 81.661) (width 1) (layer B.Cu) (net 2))
@@
   (segment (start 129.794 48.006) (end 129.794 50.038) (width 1) (layer B.Cu) (net 20))
   (segment (start 129.794 50.038) (end 130.302 50.546) (width 1) (layer B.Cu) (net 20))
-  (segment (start 130.045 50.289) (end 122.428 50.289) (width 1) (layer F.Cu) (net 20) (status 800000))
+  (segment (start 130.045 50.289) (end 122.428 50.289) (width 1) (layer F.Cu) (net 20))
   (via (at 130.302 50.546) (size 1) (drill 0.8) (layers F.Cu B.Cu) (net 20))
   (segment (start 130.302 50.546) (end 130.045 50.289) (width 1) (layer F.Cu) (net 20))
-  (segment (start 112.034 75.692) (end 106.426 75.692) (width 1) (layer B.Cu) (net 20) (status 400000))
+  (segment (start 112.034 75.692) (end 106.426 75.692) (width 1) (layer B.Cu) (net 20))
   (segment (start 106.426 75.692) (end 104.648 73.914) (width 1) (layer B.Cu) (net 20))
-  (segment (start 111.934 80.772) (end 104.648 80.772) (width 1) (layer B.Cu) (net 20) (status 400000))
-  (segment (start 104.648 70.612) (end 111.934 70.612) (width 1) (layer B.Cu) (net 20) (status 800000))
+  (segment (start 111.934 80.772) (end 104.648 80.772) (width 1) (layer B.Cu) (net 20))
+  (segment (start 104.648 70.612) (end 111.934 70.612) (width 1) (layer B.Cu) (net 20))
   (segment (start 104.648 80.772) (end 104.648 73.914) (width 1) (layer B.Cu) (net 20))
   (segment (start 104.648 73.914) (end 104.648 70.612) (width 1) (layer B.Cu) (net 20))
@@
     (connect_pads yes (clearance 1))
     (min_thickness 1)
-    (fill (arc_segments 16) (thermal_gap 0.508) (thermal_bridge_width 1.1) (smoothing fillet) (radius 3))
+    (fill yes (arc_segments 16) (thermal_gap 0.508) (thermal_bridge_width 1.1) (smoothing fillet) (radius 3))
     (polygon
       (pts
@@
     (connect_pads yes (clearance 1))
     (min_thickness 1)
-    (fill (arc_segments 16) (thermal_gap 0.508) (thermal_bridge_width 1.1) (smoothing fillet) (radius 3))
+    (fill yes (arc_segments 16) (thermal_gap 0.508) (thermal_bridge_width 1.1) (smoothing fillet) (radius 3))
     (polygon
       (pts
