File: pcb/_saved_EngineManagement.sch (KiCad schematic (older format))
At the start: 43 parts, among them K1 Temps, K5 FuelCool, K6 FuelCoolAlt, K7 Supply, U1 LM7808CT, U3 ArdinoMinPro, U5 MCP2515Shield

Commit message: Redesigned to not use VP J1939 instruments
Connections:
- net 8V: now also K7.1 (P1)
- net GND: no longer K7.1 (P1)
Changed lines of the file:
@@
 NoConn ~ 4450 7750
 NoConn ~ 4450 7950
-$Comp
-L GND #PWR09
-U 1 1 612B035D
-P 12900 5700
-F 0 "#PWR09" H 12900 5700 30  0001 C CNN
-F 1 "GND" H 12900 5630 30  0001 C CNN
-F 2 "" H 12900 5700 60  0001 C CNN
-F 3 "" H 12900 5700 60  0001 C CNN
-	1    12900 5700
-	1    0    0    -1
-$EndComp
 Text GLabel 11050 4850 2    60   Input ~ 0
 NTC1
@@
 	3900 4250 3800 4250
 Wire Wire Line
-	8500 1850 8500 1750
-Wire Wire Line
 	4850 4150 4850 4200
 Connection ~ 4400 4150
@@
 NTC3
 $Comp
-L GND #PWR010
+L GND #PWR09
 U 1 1 612B95DA
 P 5200 6700
-F 0 "#PWR010" H 5200 6700 30  0001 C CNN
+F 0 "#PWR09" H 5200 6700 30  0001 C CNN
 F 1 "GND" H 5200 6630 30  0001 C CNN
 F 2 "" H 5200 6700 60  0001 C CNN
@@
 ServiceBattery+
 Wire Wire Line
-	12900 5700 13950 5700
+	12600 5700 13950 5700
 $Comp
 L CONN_3 K1
@@
 NTC3
 $Comp
-L GND #PWR011
+L GND #PWR010
 U 1 1 612BBFFF
 P 13150 5600
-F 0 "#PWR011" H 13150 5600 30  0001 C CNN
+F 0 "#PWR010" H 13150 5600 30  0001 C CNN
 F 1 "GND" H 13150 5530 30  0001 C CNN
 F 2 "" H 13150 5600 60  0001 C CNN
@@
 Text GLabel 3400 7250 0    60   Input ~ 0
 5V150mA
+Text GLabel 12600 5700 0    60   Input ~ 0
+8V
 $EndSCHEMATC

Commit message: NTC sensors working correctly
Parts:
- R10, R11, R8: value 22K -> 4.7K
Other:
- note added: "Coolant Sensor\nWith 12V supply R23 fitted externally.\n120C == 22R\n0C = 1743R\n120C == 12*22/(1000+22)=0.25V\n80C = 12*70/1000+70)=0.78V \n50C = 12*197/(1000+197)=1.97\n20C = 12*677/(1000+677)=4.8\n11mA\n\n\n"
- note added: "Coolant Sensor\nWith 8V supply R23 at 1K\n120C == 22R\n0C = 1743R\n120C == 8*22/(1000+22)=0.17V\n80C = 8*70/1000+70)=0.52V \n50C = 8*197/1000+70)=1.3V\n8mA\n\n\n"
- note removed: "Coolant Sensor\n120C == 22R\n0C = 1743R\n120C == 8*22/(1000+22)=0.17V\n80C = 8*70/1000+70)=0.52V \n50C = 8*197/1000+70)=1.3V\n8mA\n\n\n"
Changed lines of the file:
@@
 Fuel Sensor\n0R == Empty\n190R ==  Full\nSupply 8V Use 1K, Full 1.2V empty 0v\nCurrent  max 8mA, 64mW\n
 Text Notes 8000 3600 0    60   ~ 0
-Coolant Sensor\n120C == 22R\n0C = 1743R\n120C == 8*22/(1000+22)=0.17V\n80C = 8*70/1000+70)=0.52V \n50C = 8*197/1000+70)=1.3V\n8mA\n\n\n
+Coolant Sensor\nWith 8V supply R23 at 1K\n120C == 22R\n0C = 1743R\n120C == 8*22/(1000+22)=0.17V\n80C = 8*70/1000+70)=0.52V \n50C = 8*197/1000+70)=1.3V\n8mA\n\n\n
 $Comp
 L MCP2515Shield U5
@@
 P 8950 4300
 F 0 "R8" V 9030 4300 40  0000 C CNN
-F 1 "22K" V 8957 4301 40  0000 C CNN
+F 1 "4.7K" V 8957 4301 40  0000 C CNN
 F 2 "Resistors_SMD:R_0805_HandSoldering" V 8880 4300 30  0001 C CNN
 F 3 "" H 8950 4300 30  0000 C CNN
@@
 P 9200 4300
 F 0 "R10" V 9280 4300 40  0000 C CNN
-F 1 "22K" V 9207 4301 40  0000 C CNN
+F 1 "4.7K" V 9207 4301 40  0000 C CNN
 F 2 "Resistors_SMD:R_0805_HandSoldering" V 9130 4300 30  0001 C CNN
 F 3 "" H 9200 4300 30  0000 C CNN
@@
 P 9450 4300
 F 0 "R11" V 9530 4300 40  0000 C CNN
-F 1 "22K" V 9457 4301 40  0000 C CNN
+F 1 "4.7K" V 9457 4301 40  0000 C CNN
 F 2 "Resistors_SMD:R_0805_HandSoldering" V 9380 4300 30  0001 C CNN
 F 3 "" H 9450 4300 30  0000 C CNN
@@
 Text GLabel 12600 5700 0    60   Input ~ 0
 8V
+Text Notes 9800 3600 0    60   ~ 0
+Coolant Sensor\nWith 12V supply R23 fitted externally.\n120C == 22R\n0C = 1743R\n120C == 12*22/(1000+22)=0.25V\n80C = 12*70/1000+70)=0.78V \n50C = 12*197/(1000+197)=1.97\n20C = 12*677/(1000+677)=4.8\n11mA\n\n\n
 $EndSCHEMATC
