File: pcb/EngineManagementSimpleWithMosfets.kicad_pcb (KiCad board)
At the start: 2 copper layers, 150 x 100 mm, 136 parts, among them K201 Temps, K202 FuelCool, K203 FuelCoolAlt, K204 Supply, P1 VPButtons, P11 Battery+, P2 ToEngine, P3 StarterSolenoidT30, P4 StopSolenoid, P5 12VSwitchedPower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

Commit message: After testing, fixed a number of things
Parts:
- removed the REF** at (193.8, 140.7)
- removed the REF** at (193.3, 50.0)
- removed the REF** at (53.1, 49.8)
- removed the REF** at (50.5, 142.0)
- removed the REF** at (126.2, 141.2)
- added C101: 22pF, Resistors_SMD:R_0603_HandSoldering, F.Cu at (162.3, 66.0)
- added C102: 22pF, Resistors_SMD:R_0603_HandSoldering, F.Cu at (167.4, 66.0)
- added C103: 10uF, Resistors_SMD:R_1206_HandSoldering, F.Cu at (159.8, 78.5)
- added C104: 100nF, Capacitors_SMD:C_0805_HandSoldering, F.Cu at (176.8, 81.8)
- added C105: 100nF, Capacitors_SMD:C_0805_HandSoldering, F.Cu at (186.7, 75.9)
- added D101: SMBJ30CA-TR TSV, Diodes_SMD:DO-214AB_Handsoldering, B.Cu at (189.2, 97.3)
- added D102: SMBJ30CA-TR TSV, Diodes_SMD:DO-214AB_Handsoldering, B.Cu at (189.2, 83.6)
- added P101: CanBus, Connect:bornier2, F.Cu at (185.9, 90.2)
- added R101: 10K, Resistors_SMD:R_0805_HandSoldering, F.Cu at (174.8, 84.6)
- added R220: 22K, Resistors_SMD:R_0805_HandSoldering, F.Cu at (167.8, 119.5)
- added R221: 100K, Resistors_SMD:R_0805_HandSoldering, F.Cu at (167.8, 114.7)
- added R222: 100K, Resistors_SMD:R_0805_HandSoldering, F.Cu at (173.7, 111.5)
- added REF**: 1pin, Connect:1pin, F.Cu at (51.3, 49.0)
- added REF**: 1pin, Connect:1pin, F.Cu at (51.1, 141.7)
- added REF**: 1pin, Connect:1pin, F.Cu at (193.5, 141.0)
- added REF**: 1pin, Connect:1pin, F.Cu at (193.3, 49.3)
- added U101: MCP2515, Housings_SOIC:SOIC-18W_7.5x11.6mm_Pitch1.27mm, F.Cu at (167.9, 77.0)
- added U102: TJA1050, Housings_SOIC:SOIC-8_3.9x4.9mm_Pitch1.27mm, F.Cu at (182.4, 76.2)
- added U204: LM358, Housings_DIP:DIP-8_W7.62mm_LongPads, F.Cu at (170.8, 116.0)
- added X101: 8MHz, Crystals:Resonator-2pin_w10.0mm_h5.0mm, B.Cu at (162.3, 69.3)
- C201, C202: value 10nF -> 1uF; footprint Capacitors_SMD:C_0805_HandSoldering -> Capacitors_SMD:C_1210
- D201: footprint Diodes_SMD:SOD-123 -> Diodes_SMD:D_SOD-123
- D204: footprint Diodes_SMD:D_SOD-123 -> Resistors_ThroughHole:Resistor_Horizontal_RM7mm
- R201, R202: value 47K -> 22K
- R206: value 100K -> 1K
- R3: value 10K -> 2.2K
- R6: value 2.2K -> 10K
- moved C206 69.3 mm to (159.3, 57.1), turned to 90 degrees
- moved C202 14.2 mm to (169.2, 111.5), turned to 180 degrees
- moved R206 11.8 mm to (164.2, 113.9), turned to 180 degrees
- moved D202 11.2 mm to (164.2, 116.2), turned to 0 degrees
- moved R204 9.60 mm to (184.9, 127.0), turned to 180 degrees
- moved R207 9.34 mm to (184.9, 116.1), turned to 0 degrees
- moved R205 8.93 mm to (184.9, 122.7), turned to 0 degrees
- moved C201 6.77 mm to (164.2, 118.5), turned to 180 degrees
- moved C204 6.73 mm to (184.9, 118.1), turned to 180 degrees
- moved R201 6.53 mm to (165.5, 124.6)
- moved C203 5.84 mm to (184.9, 124.7), turned to 180 degrees
- moved D201 4.90 mm to (164.2, 120.8), turned to 180 degrees
- moved R203 4.50 mm to (184.9, 120.4), turned to 180 degrees
- moved D204 3.94 mm to (158.2, 48.0), turned to 180 degrees
- moved C205 2.03 mm to (153.4, 52.3)
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Connections:
- C201 pad 1: Flywheel+ -> Net-(C201-Pad1)
- C201 pad 2: Net-(C201-Pad2) -> GND
- C202 pad 1: Flywheel- -> Net-(C202-Pad1)
- C202 pad 2: Net-(C202-Pad2) -> GND
- D201 pad 1: Net-(D201-Pad1) -> Net-(C201-Pad1)
- D201 pad 2: 5V150mA -> GND
- D202 pad 2: Net-(D201-Pad1) -> Net-(C201-Pad1)
- K204 pad 1: 8V -> GND
- R201 pad 1: Net-(C201-Pad2) -> Flywheel+
- R201 pad 2: Net-(D201-Pad1) -> Net-(C201-Pad1)
- R202 pad 1: Net-(C202-Pad2) -> Flywheel-
- R206 pad 1: Net-(D201-Pad1) -> Net-(C201-Pad1)
- U203 pad 5: Net-(D201-Pad1) -> RPMPulse
Routing:
- net GND: track 793.2 -> 1128.0 mm, vias 11 -> 10
- net 5V150mA: track 111.1 -> 178.2 mm, vias 5 -> 4
- net 8V: track 166.0 -> 121.9 mm, vias 4 -> 3
- net Net-(C201-Pad1): track 0.00 -> 27.0 mm
- net Net-(D201-Pad1): track 25.6 -> 0.00 mm, vias 1 -> 0
- net RPMPulse: track 0.00 -> 21.3 mm
- net Net-(D101-Pad2): track 0.00 -> 19.5 mm, vias 0 -> 1
- net Net-(U101-Pad1): track 0.00 -> 16.7 mm
- net 12vSwitched: track 330.1 -> 313.4 mm, vias 6 -> 5
- net Net-(D102-Pad2): track 0.00 -> 13.3 mm, vias 0 -> 1
- net ServiceBattery+: track 9.92 -> 22.8 mm
- net CANCS: track 44.9 -> 56.7 mm, vias 2 -> 3
- net Net-(U101-Pad2): track 0.00 -> 11.2 mm
- net Net-(C202-Pad1): track 0.00 -> 11.0 mm
- net Net-(C204-Pad1): track 39.7 -> 29.4 mm
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Other:
- net class Default: via_dia 1.5 -> 1.2
