File: pcb/EngineManagementSimpleWithMosfets.sch (KiCad schematic (older format))
At the start: 100 parts, among them P1 VPButtons, P10 VP ButtonPlug, P2 ToEngine, P3 StarterSolenoidT30, P4 StopSolenoid, P5 12VSwitchedPower, P6 GlowPlugs, P8 VP EnginePlug, P9 VP MultiLinkPlug, Q1 BC807, Q11 BS250P, Q13 BS250P, Q15 BS250P, Q2 BS170, Q3 SI7137, Q4 SI7137, Q5 BC807, Q6 BC807, Q7 SI7137, Q8 SI7137, Q9 SI7137, SW1 ON/OFF, SW2 Start, SW3 Stop, SW4 Glow, SW5 Neutral, U1 LM358, U2 Tachometer, U3 WaterTemp, U4 NCP1117ST50T3G, U5 Max16054

Commit message: After testing, fixed a number of things
Parts:
- added P11: Battery+, Divers:CrimpBlade, symbol CONN_1
- added P7: 0v, Divers:CrimpBlade, symbol CONN_1
- R3: value 10K -> 2.2K
- R6: value 2.2K -> 10K
Connections:
- net Battery+: now also P11.1
- net GND: now also P7.1
Changed lines of the file:
@@
 P 2850 7950
 F 0 "R3" H 2930 7950 40  0000 C CNN
-F 1 "10K" V 2857 7951 40  0000 C CNN
+F 1 "2.2K" V 2857 7951 40  0000 C CNN
 F 2 "Resistors_SMD:R_0805_HandSoldering" V 2780 7950 30  0001 C CNN
 F 3 "" H 2850 7950 30  0000 C CNN
@@
 P 3300 8250
 F 0 "R6" H 3380 8250 40  0000 C CNN
-F 1 "2.2K" V 3307 8251 40  0000 C CNN
+F 1 "10K" V 3307 8251 40  0000 C CNN
 F 2 "Resistors_SMD:R_0805_HandSoldering" V 3230 8250 30  0001 C CNN
 F 3 "" H 3300 8250 30  0000 C CNN
@@
 F1 "EngineManagement.sch" 60
 $EndSheet
+$Comp
+L CONN_1 P11
+U 1 1 6155F876
+P 4500 600
+F 0 "P11" H 4580 600 40  0000 L CNN
+F 1 "Battery+" H 4500 655 30  0000 C CNN
+F 2 "Divers:CrimpBlade" H 4500 600 60  0001 C CNN
+F 3 "" H 4500 600 60  0001 C CNN
+	1    4500 600
+	1    0    0    -1
+$EndComp
+Wire Wire Line
+	4350 600  4300 600
+Wire Wire Line
+	4300 600  4300 750
+Connection ~ 4300 750
+$Comp
+L CONN_1 P7
+U 1 1 615600EB
+P 4250 1200
+F 0 "P7" H 4330 1200 40  0000 L CNN
+F 1 "0v" H 4250 1255 30  0000 C CNN
+F 2 "Divers:CrimpBlade" H 4250 1200 60  0001 C CNN
+F 3 "" H 4250 1200 60  0001 C CNN
+	1    4250 1200
+	-1   0    0    1
+$EndComp
+Wire Wire Line
+	4400 1200 4750 1200
+Wire Wire Line
+	4750 1200 4750 1300
+Wire Wire Line
+	4750 1300 5000 1300
+Connection ~ 5000 1300
 $EndSCHEMATC
