File: pcb/EngineManagement.kicad_pcb (KiCad board)
At the start: 2 copper layers, 97 x 56.1 mm, 47 parts, among them K1 Temps, K5 FuelCool, K6 FuelCoolAlt, K7 Supply, U1 LM7808CT, U3 ArdinoMinPro, U5 MCP2515Shield

Commit message: Added pdfs for reference
Parts:
- moved REF** 8.13 mm to (100.8, 94.2)
- moved REF** 8.13 mm to (100.8, 48.8)
- moved REF** 5.61 mm to (191.3, 94.2)
- moved REF** 5.59 mm to (191.5, 48.5)
Other:
- board text added: "0v"
- board text added: "12v In"
- board text added: "8v Out"
- board text added: "Alternatore B+"
- board text added: "Coolant Sensor +"
- board text added: "Flywheel +"
- board text added: "Flywheel -"
- board text added: "Fuel Level +"
- board text added: "NCT1"
- board text added: "NCT2"
- board text added: "NCT3"
- board text added: "Service Battery +"
Changed lines of the file:
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@@
     (links 83)
     (no_connects 0)
-    (area 96.952999 42.850999 194.131001 99.135001)
+    (area 39.017498 13.807691 195.426001 272.896001)
     (thickness 1.6)
-    (drawings 20)
+    (drawings 33)
     (tracks 277)
     (zones 0)
@@
     (pad_drill 0.762)
     (pad_to_mask_clearance 0.2)
-    (aux_axis_origin 104.394 142.494)
+    (aux_axis_origin 96.774 99.568)
     (grid_origin 97.79 42.164)
     (visible_elements FFFFFF7F)
@@
   )
   (module Connect:1pin (layer F.Cu)
-    (at 185.928 48.514)
+    (at 191.516 48.514)
     (descr "module 1 pin (ou trou mecanique de percage)")
     (tags DEV)
@@
   )
   (module Connect:1pin (layer F.Cu)
-    (at 185.674 93.726)
+    (at 191.262 94.234)
     (descr "module 1 pin (ou trou mecanique de percage)")
     (tags DEV)
@@
   )
   (module Connect:1pin (layer F.Cu)
-    (at 108.966 94.234)
+    (at 100.838 94.234)
     (descr "module 1 pin (ou trou mecanique de percage)")
     (tags DEV)
@@
   )
   (module Connect:1pin (layer F.Cu)
-    (at 108.966 48.768)
+    (at 100.838 48.768)
     (descr "module 1 pin (ou trou mecanique de percage)")
     (tags DEV)
@@
     (fp_circle (center 0 0) (end 0 -2.286) (layer F.SilkS) (width 0.15))
     (pad 1 thru_hole circle (at 0 0) (size 4.064 4.064) (drill 3.048) (layers *.Cu *.Mask))
+  )
+  (gr_text "Flywheel -" (at 89.408 83.312) (layer Dwgs.User)
+    (effects (font (size 1.5 1.5) (thickness 0.3)))
+  )
+  (gr_text "Flywheel +" (at 88.646 77.47) (layer Dwgs.User)
+    (effects (font (size 1.5 1.5) (thickness 0.3)))
+  )
+  (gr_text "Alternatore B+" (at 87.376 72.898) (layer Dwgs.User)
+    (effects (font (size 1.5 1.5) (thickness 0.3)))
+  )
+  (gr_text "Service Battery +" (at 86.106 68.072) (layer Dwgs.User)
+    (effects (font (size 1.5 1.5) (thickness 0.3)))
+  )
+  (gr_text "12v In" (at 89.154 62.992) (layer Dwgs.User)
+    (effects (font (size 1.5 1.5) (thickness 0.3)))
+  )
+  (gr_text "8v Out" (at 89.662 57.404) (layer Dwgs.User)
+    (effects (font (size 1.5 1.5) (thickness 0.3)))
+  )
+  (gr_text NCT3 (at 198.628 58.928) (layer Dwgs.User)
+    (effects (font (size 1.5 1.5) (thickness 0.3)))
+  )
+  (gr_text NCT2 (at 198.628 64.77) (layer Dwgs.User)
+    (effects (font (size 1.5 1.5) (thickness 0.3)))
+  )
+  (gr_text NCT1 (at 198.628 69.596) (layer Dwgs.User)
+    (effects (font (size 1.5 1.5) (thickness 0.3)))
+  )
+  (gr_text 0v (at 197.104 75.438) (layer Dwgs.User)
+    (effects (font (size 1.5 1.5) (thickness 0.3)))
+  )
+  (gr_text "Fuel Level +" (at 202.946 80.01) (layer Dwgs.User)
+    (effects (font (size 1.5 1.5) (thickness 0.3)))
+  )
+  (gr_text "Coolant Sensor +" (at 205.74 84.836) (layer Dwgs.User)
+    (effects (font (size 1.5 1.5) (thickness 0.3)))
+  )
+  (dimension 77.216 (width 0.3) (layer Dwgs.User)
+    (gr_text "77.216 mm" (at 147.574 29.384) (layer Dwgs.User)
+      (effects (font (size 1.5 1.5) (thickness 0.3)))
+    )
+    (feature1 (pts (xy 186.182 42.926) (xy 186.182 28.034)))
+    (feature2 (pts (xy 108.966 42.926) (xy 108.966 28.034)))
+    (crossbar (pts (xy 108.966 30.734) (xy 186.182 30.734)))
+    (arrow1a (pts (xy 186.182 30.734) (xy 185.055496 31.320421)))
+    (arrow1b (pts (xy 186.182 30.734) (xy 185.055496 30.147579)))
+    (arrow2a (pts (xy 108.966 30.734) (xy 110.092504 31.320421)))
+    (arrow2b (pts (xy 108.966 30.734) (xy 110.092504 30.147579)))
   )
   (gr_line (start 195.326 94.234) (end 195.326 92.202) (angle 90) (layer Dwgs.User) (width 0.2))
@@
   (segment (start 116.335 59.439) (end 119.888 59.439) (width 1) (layer F.Cu) (net 1))
   (segment (start 129.032 59.69) (end 110.998 59.69) (width 1) (layer B.Cu) (net 2))
-  (segment (start 110.998 59.69) (end 108.966 57.658) (width 1) (layer B.Cu) (net 2) (status 800000))
+  (segment (start 110.998 59.69) (end 108.966 57.658) (width 1) (layer B.Cu) (net 2))
   (segment (start 147.574 56.134) (end 152.908 56.134) (width 1) (layer B.Cu) (net 2))
   (segment (start 177.419 81.661) (end 180.133 81.661) (width 1) (layer B.Cu) (net 2))
@@
   (segment (start 129.794 48.006) (end 129.794 50.038) (width 1) (layer B.Cu) (net 20))
   (segment (start 129.794 50.038) (end 130.302 50.546) (width 1) (layer B.Cu) (net 20))
-  (segment (start 130.045 50.289) (end 122.428 50.289) (width 1) (layer F.Cu) (net 20) (status 800000))
+  (segment (start 130.045 50.289) (end 122.428 50.289) (width 1) (layer F.Cu) (net 20))
   (via (at 130.302 50.546) (size 1) (drill 0.8) (layers F.Cu B.Cu) (net 20))
   (segment (start 130.302 50.546) (end 130.045 50.289) (width 1) (layer F.Cu) (net 20))
-  (segment (start 112.034 75.692) (end 106.426 75.692) (width 1) (layer B.Cu) (net 20) (status 400000))
+  (segment (start 112.034 75.692) (end 106.426 75.692) (width 1) (layer B.Cu) (net 20))
   (segment (start 106.426 75.692) (end 104.648 73.914) (width 1) (layer B.Cu) (net 20))
-  (segment (start 111.934 80.772) (end 104.648 80.772) (width 1) (layer B.Cu) (net 20) (status 400000))
-  (segment (start 104.648 70.612) (end 111.934 70.612) (width 1) (layer B.Cu) (net 20) (status 800000))
+  (segment (start 111.934 80.772) (end 104.648 80.772) (width 1) (layer B.Cu) (net 20))
+  (segment (start 104.648 70.612) (end 111.934 70.612) (width 1) (layer B.Cu) (net 20))
   (segment (start 104.648 80.772) (end 104.648 73.914) (width 1) (layer B.Cu) (net 20))
   (segment (start 104.648 73.914) (end 104.648 70.612) (width 1) (layer B.Cu) (net 20))
@@
     (connect_pads yes (clearance 1))
     (min_thickness 1)
-    (fill (arc_segments 16) (thermal_gap 0.508) (thermal_bridge_width 1.1) (smoothing fillet) (radius 3))
+    (fill yes (arc_segments 16) (thermal_gap 0.508) (thermal_bridge_width 1.1) (smoothing fillet) (radius 3))
     (polygon
       (pts
@@
     (connect_pads yes (clearance 1))
     (min_thickness 1)
-    (fill (arc_segments 16) (thermal_gap 0.508) (thermal_bridge_width 1.1) (smoothing fillet) (radius 3))
+    (fill yes (arc_segments 16) (thermal_gap 0.508) (thermal_bridge_width 1.1) (smoothing fillet) (radius 3))
     (polygon
       (pts
@@
       )
     )
+  )
+  (zone (net 0) (net_name "") (layer B.Cu) (hatch edge 0.508)
+    (connect_pads (clearance 1))
+    (min_thickness 1)
+    (keepout (tracks allowed) (vias allowed) (copperpour not_allowed))
+    (fill (arc_segments 16) (thermal_gap 0.508) (thermal_bridge_width 1.1))
+    (polygon
+      (pts
+        (xy 168.656 75.438) (xy 168.656 93.726) (xy 144.526 93.726) (xy 144.526 75.438)
+      )
+    )
+  )
+  (zone (net 0) (net_name "") (layer B.Cu) (hatch edge 0.508)
+    (connect_pads (clearance 1))
+    (min_thickness 1)
+    (keepout (tracks allowed) (vias allowed) (copperpour not_allowed))
+    (fill (arc_segments 16) (thermal_gap 0.508) (thermal_bridge_width 1.1))
+    (polygon
+      (pts
+        (xy 144.272 75.438) (xy 144.272 75.184) (xy 144.526 75.184) (xy 144.526 75.438)
+      )
+    )
+  )
+  (zone (net 0) (net_name "") (layer F.Cu) (hatch edge 0.508)
+    (connect_pads (clearance 1))
+    (min_thickness 1)
+    (keepout (tracks allowed) (vias allowed) (copperpour not_allowed))
+    (fill (arc_segments 16) (thermal_gap 0.508) (thermal_bridge_width 1.1))
+    (polygon
+      (pts
+        (xy 168.656 94.234) (xy 144.526 94.234) (xy 144.526 75.184) (xy 168.656 75.184)
+      )
+    )

Commit message: After testing, fixed a number of things
Parts:
- removed C1, C10, C12, C13, C3, C4, C5, C6: 10nF, Capacitors_SMD:C_0805_HandSoldering
- removed C2: 100uF, Capacitors_ThroughHole:C_Radial_D8_L11.5_P3.5
- removed C7, C8, C9: 1nF, Capacitors_SMD:C_0805_HandSoldering
- removed D1: SMBJ30CA-TR TSV, Diodes_SMD:DO-214AB_Handsoldering
- removed D3, D5, D6: 1N5819, Resistors_ThroughHole:Resistor_Horizontal_RM7mm
- removed K1: Temps, Connect:bornier3
- removed K5: FuelCool, Connect:bornier3
- removed K6: FuelCoolAlt, Connect:bornier3
- removed K7: Supply, Connect:bornier3
- removed R1, R25, R27: 1M, Resistors_SMD:R_0805_HandSoldering
- removed R10, R11, R8: 22K, Resistors_SMD:R_0805_HandSoldering
- removed R2, R21, R22, R6, R7: 100K, Resistors_SMD:R_0805_HandSoldering
- removed R23, R24: 1K, Resistors_SMD:R_0805_HandSoldering
- removed R26, R28, R30: 470K, Resistors_SMD:R_0805_HandSoldering
- removed R3, R4: 47K, Resistors_SMD:R_0805_HandSoldering
- removed R5: 10K, Resistors_SMD:R_0805_HandSoldering
- removed the REF** at (191.5, 48.5)
- removed the REF** at (191.3, 94.2)
- removed the REF** at (100.8, 94.2)
- removed the REF** at (100.8, 48.8)
- removed TH1: 500mA Thermistor, Resistors_ThroughHole:Resistor_Horizontal_RM7mm
- removed U1: LM7808CT, TO_SOT_Packages_SMD:TO-263-3Lead
- removed U3: ArdinoMinPro, Divers:ArduinoProMini
- removed U5: MCP2515Shield, Divers:MCP2515Board
- added C101: 22pF, Resistors_SMD:R_0603_HandSoldering, F.Cu at (119.9, 87.9)
- added C102: 22pF, Resistors_SMD:R_0603_HandSoldering, F.Cu at (119.9, 85.3)
- added C103: 10uF, Resistors_SMD:R_1206_HandSoldering, F.Cu at (131.8, 71.9)
- added C104: 100nF, Capacitors_SMD:C_0805_HandSoldering, F.Cu at (119.9, 71.9)
- added C105: 100nF, Capacitors_SMD:C_0805_HandSoldering, F.Cu at (132.3, 74.7)
- added C201: 1uF, Capacitors_SMD:C_1210, B.Cu at (165.9, 80.8)
- added C202: 1uF, Capacitors_SMD:C_1210, B.Cu at (165.6, 91.2)
- added C203: 1nF, Capacitors_SMD:C_0805_HandSoldering, B.Cu at (109.5, 56.1)
- added C204: 1nF, Capacitors_SMD:C_0805_HandSoldering, B.Cu at (103.9, 65.5)
- added C205: 100uF, Capacitors_ThroughHole:C_Radial_D8_L11.5_P3.5, F.Cu at (118.6, 60.2)
- added C206: 10nF, Capacitors_SMD:C_0805_HandSoldering, B.Cu at (165.1, 63.0)
- added C207: 10nF, Capacitors_SMD:C_0805_HandSoldering, B.Cu at (185.9, 67.6)
- added C208: 10nF, Capacitors_SMD:C_0805_HandSoldering, B.Cu at (185.9, 72.6)
- added C209: 10nF, Capacitors_SMD:C_0805_HandSoldering, B.Cu at (185.7, 61.7)
- added C210: 10nF, Capacitors_SMD:C_0805_HandSoldering, B.Cu at (185.7, 56.9)
- added C211: 10nF, Capacitors_SMD:C_0805_HandSoldering, B.Cu at (185.4, 50.0)
- added C212: 1nF, Capacitors_SMD:C_0805_HandSoldering, B.Cu at (173.7, 79.0)
- added D101: SMBJ30CA-TR TSV, Diodes_SMD:DO-214AB_Handsoldering, B.Cu at (105.9, 75.2)
- added D102: SMBJ30CA-TR TSV, Diodes_SMD:DO-214AB_Handsoldering, B.Cu at (105.7, 90.7)
- added D201: 1N5819, Diodes_SMD:D_SOD-123, B.Cu at (175.0, 82.8)
- added D202: 1N5819, Diodes_SMD:D_SOD-123, B.Cu at (175.0, 88.1)
- added D203: SMBJ30CA-TR TSV, Diodes_SMD:DO-214AB_Handsoldering, B.Cu at (111.8, 68.3)
- added D204: 1N5819, Resistors_ThroughHole:Resistor_Horizontal_RM7mm, F.Cu at (127.3, 67.8)
- added K201: Temps, Connect:bornier3, F.Cu at (182.9, 56.1)
- added K202: FuelCool, Connect:bornier3, F.Cu at (182.9, 86.6)
- added K203: FuelCoolAlt, Connect:bornier3, F.Cu at (182.9, 71.4)
- added K204: Supply, Connect:bornier3, F.Cu at (104.4, 55.6)
- added P101: CanBus, Connect:bornier2, F.Cu at (110.0, 83.6)
- added R101: 10K, Resistors_SMD:R_0805_HandSoldering, F.Cu at (138.2, 78.0)
- added R201: 22K, Resistors_SMD:R_0805_HandSoldering, B.Cu at (177.3, 87.9)
- added R202: 22K, Resistors_SMD:R_0805_HandSoldering, B.Cu at (175.3, 92.7)
- added R203: 1M, Resistors_SMD:R_0805_HandSoldering, B.Cu at (109.5, 61.0)
- added R204: 1M, Resistors_SMD:R_0805_HandSoldering, B.Cu at (109.5, 53.6)
- added R205: 470K, Resistors_SMD:R_0805_HandSoldering, B.Cu at (113.3, 57.7)
- added R206: 1K, Resistors_SMD:R_0805_HandSoldering, B.Cu at (172.5, 82.8)
- added R207: 470K, Resistors_SMD:R_0805_HandSoldering, B.Cu at (109.5, 58.7)
- added R208: 100K, Resistors_SMD:R_0805_HandSoldering, B.Cu at (175.5, 46.2)
- added R209: 100K, Resistors_SMD:R_0805_HandSoldering, B.Cu at (175.5, 54.1)
- added R210: 100K, Resistors_SMD:R_0805_HandSoldering, B.Cu at (175.5, 59.9)
- added R211: 100K, Resistors_SMD:R_0805_HandSoldering, B.Cu at (175.3, 72.9)
- added R212: 100K, Resistors_SMD:R_0805_HandSoldering, B.Cu at (175.3, 64.8)
- added R213: 1K, Resistors_SMD:R_0805_HandSoldering, B.Cu at (175.3, 67.3)
- added R214: 1K, Resistors_SMD:R_0805_HandSoldering, B.Cu at (175.3, 70.6)
- added R215: 4.7K, Resistors_SMD:R_0805_HandSoldering, B.Cu at (175.5, 57.7)
- added R216: 4.7K, Resistors_SMD:R_0805_HandSoldering, B.Cu at (175.5, 51.8)
- added R217: 4.7K, Resistors_SMD:R_0805_HandSoldering, B.Cu at (175.5, 48.5)
- added R218: 470K, Resistors_SMD:R_0805_HandSoldering, B.Cu at (177.3, 80.0)
- added R219: 1M, Resistors_SMD:R_0805_HandSoldering, B.Cu at (179.8, 80.0)
- added R220: 22K, Resistors_SMD:R_0805_HandSoldering, B.Cu at (172.5, 88.1)
- added R221: 100K, Resistors_SMD:R_0805_HandSoldering, B.Cu at (169.9, 92.7)
- added R222: 100K, Resistors_SMD:R_0805_HandSoldering, B.Cu at (165.9, 85.9)
- added REF**: 1pin, Connect:1pin, F.Cu at (190.8, 95.5)
- added REF**: 1pin, Connect:1pin, F.Cu at (191.0, 46.2)
- added REF**: 1pin, Connect:1pin, F.Cu at (100.8, 46.2)
- added REF**: 1pin, Connect:1pin, F.Cu at (100.8, 95.8)
- added TH201: 500mA Thermistor, Resistors_ThroughHole:Resistor_Horizontal_RM7mm, F.Cu at (117.3, 49.3)
- added U101: MCP2515, Housings_SOIC:SOIC-18W_7.5x11.6mm_Pitch1.27mm, F.Cu at (130.8, 83.6)
- added U102: TJA1050, Housings_SOIC:SOIC-8_3.9x4.9mm_Pitch1.27mm, F.Cu at (119.6, 76.2)
- added U201: MCP2515Shield, Divers:MCP2515Board, F.Cu at (142.5, 98.0)
- added U202: LM7808CT, TO_SOT_Packages_SMD:TO-263-3Lead, F.Cu at (127.3, 58.4)
- added U203: ArdinoMinPro, Divers:ArduinoProMini, F.Cu at (160.0, 63.2)
- added U204: LM358, Housings_DIP:DIP-8_W7.62mm_LongPads, F.Cu at (169.4, 89.4)
- added X101: 8MHz, Crystals:Resonator-2pin_w10.0mm_h5.0mm, B.Cu at (121.4, 89.2)
Routing:
- net GND: track 371.0 -> 558.9 mm, vias 1 -> 3
- net Net-(C204-Pad1): track 0.00 -> 72.8 mm, vias 0 -> 2
- net Net-(C7-Pad1): track 72.3 -> 0.00 mm, vias 2 -> 0
- net RPMPulse: track 0.00 -> 66.4 mm, vias 0 -> 1
- net Net-(R2-Pad1): track 66.3 -> 0.00 mm, vias 2 -> 0
- net 12V: track 56.6 -> 0.00 mm, vias 1 -> 0
- net Net-(C203-Pad1): track 0.00 -> 52.0 mm
- net Net-(C212-Pad1): track 0.00 -> 50.4 mm, vias 0 -> 2
- net Net-(C9-Pad1): track 50.3 -> 0.00 mm
- net Net-(R212-Pad1): track 0.00 -> 50.1 mm, vias 0 -> 2
- net 8V: track 104.8 -> 59.8 mm, vias 3 -> 2
- net Net-(R209-Pad1): track 0.00 -> 39.5 mm
- net Net-(R210-Pad1): track 0.00 -> 39.2 mm
- net Net-(C2-Pad1): track 39.0 -> 0.00 mm
- net Net-(D5-Pad1): track 37.4 -> 0.00 mm, vias 1 -> 0
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Other:
- net class Default: via_dia 1 -> 1.5; via_drill 0.8 -> 0.7
- board text added: "12v"
- board text added: "AltB+"
- board text added: "Fly+"
- board text added: "Fly-"
- board text added: "Fuel"
- board text added: "Temp"
- board text removed: "12v In"
- board text removed: "8v Out"
- board text removed: "Alternatore B+"
- board text removed: "Coolant Sensor +"
- board text removed: "Flywheel +"
- board text removed: "Flywheel -"
- board text removed: "Fuel Level +"
