File: pcb/MosfetSwitch.sch (KiCad schematic (older format))
At the start: 102 parts, among them P1 VPButtons, P10 VP ButtonPlug, P11 Battery+, P2 ToEngine, P3 StarterSolenoidT30, P4 StopSolenoid, P5 12VSwitchedPower, P6 GlowPlugs, P7 0v, P8 VP EnginePlug, P9 VP MultiLinkPlug, Q1 BC807, Q11 BS250P, Q13 BS250P, Q15 BS250P, Q2 BS170, Q3 SI7137, Q4 SI7137, Q5 BC807, Q6 BC807, Q7 SI7137, Q8 SI7137, Q9 SI7137, SW1 ON/OFF, SW2 Start, SW3 Stop, SW4 Glow, SW5 Neutral, U1 LM358, U2 Tachometer, U3 WaterTemp, U4 NCP1117ST50T3G, U5 Max16054

Commit message: After testing, fixed a number of things
Parts:
- R3: value 10K -> 2.2K
- R6: value 2.2K -> 10K
Changed lines of the file:
@@
 P 2850 7950
 F 0 "R3" H 2930 7950 40  0000 C CNN
-F 1 "10K" V 2857 7951 40  0000 C CNN
+F 1 "2.2K" V 2857 7951 40  0000 C CNN
 F 2 "Resistors_SMD:R_0805_HandSoldering" V 2780 7950 30  0001 C CNN
 F 3 "" H 2850 7950 30  0000 C CNN
@@
 P 3300 8250
 F 0 "R6" H 3380 8250 40  0000 C CNN
-F 1 "2.2K" V 3307 8251 40  0000 C CNN
+F 1 "10K" V 3307 8251 40  0000 C CNN
 F 2 "Resistors_SMD:R_0805_HandSoldering" V 3230 8250 30  0001 C CNN
 F 3 "" H 3300 8250 30  0000 C CNN
@@
 	5300 850  5300 750
 Connection ~ 5300 750
-$Sheet
-S 11300 8500 4150 1250
-U 615569F0
-F0 "EngineManagement" 60
-F1 "EngineManagement.sch" 60
-$EndSheet
 $Comp
 L CONN_1 P11

Commit message: Istalled working version, all working, may need some adjustment on messages
Parts:
- removed C1: 10nF, Capacitors_SMD:C_0805_HandSoldering, symbol C
- removed C2, C3: 10uF, Capacitors_ThroughHole:C_Radial_D8_L11.5_P3.5, symbol CAPAPOL
- removed D10: 10A 600V, Diodes_ThroughHole:Diode_P600_Vertical_AnodeUp, symbol DIODE
- removed D11, D19, D6: SMBJ30CA-TR TSV, Diodes_SMD:DO-214AB_Handsoldering, symbol DIODE
- removed D12, D16: ZENER, Diodes_SMD:D_SOD-123, symbol ZENER
- removed D14: PowerOn, Resistors_SMD:R_0805_HandSoldering, symbol LED
- removed D17: 10V Zeener, Diodes_SMD:D_SOD-123, symbol ZENER
- removed D2: ChargeWarn, Resistors_SMD:R_0805_HandSoldering, symbol LED
- removed D20: 1N4001, Diodes_SMD:D_SOD-123, symbol DIODE
- removed D3: 10A100V, Resistors_ThroughHole:Resistor_Horizontal_RM7mm, symbol DIODE
- removed D4: TempWarn, Resistors_SMD:R_0805_HandSoldering, symbol LED
- removed D5: OilWarn, Resistors_SMD:R_0805_HandSoldering, symbol LED
- removed D9: 1A 40V, Diodes_SMD:DO-214AB, symbol DIODE
- removed F1: FUSE 5A, Divers:BladeFuse-CarType, symbol FUSE
- removed F2: FUSE 30A, Divers:BladeFuse-CarType, symbol FUSE
- removed F3: 6A Breaker, symbol FUSE
- removed F4, F5: 6A breaker, symbol FUSE
- removed F6, F8: FUSE 40A, Divers:BladeFuse-CarType, symbol FUSE
- removed F7: FUSE 15A, Divers:BladeFuse-CarType, symbol FUSE
- removed P1: VPButtons, Connect:bornier5, symbol CONN_5
- removed P10: VP ButtonPlug, symbol CONN_6
- removed P8: VP EnginePlug, symbol CONN_8
- removed P9: VP MultiLinkPlug, symbol CONN_6
- removed Q1, Q5, Q6: BC807, TO_SOT_Packages_SMD:SOT-23_Handsoldering, symbol PNP
- removed Q13, Q15: BS250P, TO_SOT_Packages_SMD:SOT-23_Handsoldering, symbol MOSFET_P
- removed Q2: BS170, TO_SOT_Packages_SMD:SOT-23_Handsoldering, symbol MOS_N
- removed Q8: SI7137, Divers:Si7137PowerPak, symbol MOSFET_P
- removed R25, R8, R9: 10K, Resistors_SMD:R_0805_HandSoldering, symbol R
- removed R26: 1K, Resistors_SMD:R_0805_HandSoldering, symbol R
- removed R27, R28, R3: 2.2K, Resistors_SMD:R_0805_HandSoldering, symbol R
- removed R31: 100R, Resistors_SMD:R_0805_HandSoldering, symbol R
- removed R34, R35: 220R, Resistors_SMD:R_0805_HandSoldering, symbol R
- removed RV1: 20K, Potentiometers:Potentiometer_Bourns_3296W_3-8Zoll_Inline_ScrewUp, symbol POT
- removed SP1: Buzzer, symbol SPEAKER
- removed SW1: ON/OFF, symbol SW_PUSH
- removed SW2: Start, symbol SW_PUSH
- removed SW3: Stop, symbol SW_PUSH
- removed SW4: Glow, symbol SW_PUSH
- removed SW5: Neutral, symbol SPST
- removed TH1: THERMISTOR, Resistors_ThroughHole:Resistor_Horizontal_RM7mm, symbol THERMISTOR
- removed U1: LM358, Housings_DIP:DIP-8_W7.62mm_LongPads, symbol LM358
- removed U2: Tachometer, symbol Tachometer
- removed U3: WaterTemp, symbol Tachometer
- removed U4: NCP1117ST50T3G, TO_SOT_Packages_SMD:SOT-223-3Lead_TabPin2, symbol NCP1117ST50T3G
- removed U5: Max16054, TO_SOT_Packages_SMD:SOT-23-6_Handsoldering, symbol Max16054
- added D13, D14, D15, D28, D29, D30: 1N4001, Resistors_ThroughHole:Resistor_Horizontal_RM7mm, symbol DIODE
- added D16, D17, D2: SMBJ30CA-TR TSV, Diodes_SMD:DO-214AB_Handsoldering, symbol DIODE
- added D19, D20, D21, D4, D5: ZENER, Diodes_SMD:D_SOD-123, symbol ZENER
- added D24: 1N4001, Diodes_SMD:D_SOD-123, symbol DIODE
- added P10: CH5In, Divers:CrimpBlade, symbol CONN_1
- added P12: Ch6Out, Divers:CrimpBlade, symbol CONN_1
- added P13: Ch5Out, Divers:CrimpBlade, symbol CONN_1
- added P14: Ch4Out, Divers:CrimpBlade, symbol CONN_1
- added P15, P16, P17, P18: hole, Connect:1pin, symbol CONN_1
- added P2: 0v, Divers:CrimpBlade, symbol CONN_1
- added P4: CH2In, Divers:CrimpBlade, symbol CONN_1
- added P9: CH6In, Divers:CrimpBlade, symbol CONN_1
- added Q1: SI7137, Divers:Si7137PowerPak, symbol MOSFET_P
- added Q10, Q12, Q2, Q4, Q6, Q8: BC817-40, TO_SOT_Packages_SMD:SOT-23, symbol BC817-40
- added R13, R15: 10K, Resistors_SMD:R_0805_HandSoldering, symbol R
- D18: value 5A 600V -> SMBJ30CA-TR TSV; footprint Diodes_ThroughHole:Diode_P600_Vertical_AnodeUp -> Diodes_SMD:DO-214AB_Handsoldering
- D7: value 5A 600V -> 1N4001; footprint Diodes_ThroughHole:Diode_P600_Vertical_AnodeUp -> Diodes_SMD:D_SOD-123
- D8: value 10A 600V -> 1N4001; footprint Diodes_ThroughHole:Diode_P600_Vertical_KathodeUp -> Diodes_SMD:D_SOD-123
- P1: renamed from P2; value ToEngine -> ToSwitches
- P11: value Battery+ -> CH4In
- P3: value StarterSolenoidT30 -> CH3In
- P5: value 12VSwitchedPower -> CH1In
- P6: value GlowPlugs -> Ch3Out
- P7: value 0v -> Ch2Out
- P8: renamed from P4; value StopSolenoid -> Ch1Out
- Q11: value BS250P -> SI7137; footprint TO_SOT_Packages_SMD:SOT-23_Handsoldering -> Divers:Si7137PowerPak
- R1: value 100R -> 10K
- R10: value 220R -> 470R
- R11, R22, R23: value 1K -> 470R
- R12: value 10M -> 470R
- R14, R16, R19: value 1K -> 10K
- R18, R20: value 2.2K -> 10K
- R2: value 330R -> 10K
- R24: value 100R -> 470R
- R3: renamed from R15; value 100R -> 10K
- R7: value 10R -> 10K; footprint Resistors_ThroughHole:Resistor_Horizontal_RM20mm -> Resistors_SMD:R_0805_HandSoldering
- R8: renamed from R13; value 1K -> 10K
- R9: renamed from R33; value 220R -> 10K
- renumbered D13 to D3, D15 to D6, D21 to D9, Q4 to Q5
Connections:
- net labels added: CH1_SWITCH, CH2_SWITCH, CH3_SWITCH, CH4_SWITCH, CH5_SWITCH, CH6_SWITCH
- net labels removed: 0V, 0V-SB, 12vSwitched, AccDimmer-W, AlternatorExcitation, Battery+, Buzzer, Buzzer-?, CanH-Y/W, CanL-Y/GR, CoolantSensorVP-LBN, CoolantTemp, Enable, EngineRoomFan, ExcitationVP, Flywheel+, Flywheel-, FlywheelVP+-GR/SB, FlywheelVP--GR, GlowBtn, GlowPlugs, KeelController, MultiLink0V-SB, MultiLink12V-R, OilPressureVP-SB, OilSwitch, OnOff-R, OnOffBtn, STOP-VO, Start-Y, StartBtn, StarterSolenoidT30, StopBtn, StopSolenoid, StopSolenoid-VO, WindlassController
- wire segments 254 -> 128
- no-connect marks 3 -> 4
Other:
- note removed: "10A"
- note removed: "40A"
- note removed: "8A"
- note removed: "Cockpit"
- note removed: "ControlBoard"
- note removed: "SB,BL,BL,BL\n"
- note removed: "SB,BL,BL,Y\n"
- note removed: "SB,BL,BL\n"
- note removed: "SB,BL,R\n"
- note removed: "SB,BL,W\n"
- note removed: "SB,BL,Y\n"
- note removed: "SB,SB,BL\n"
- note removed: "SB,SB,R\n"
- note removed: "SB,SB,SB,BL\n"
- note removed: "SB,SB,SB,R\n"
- note removed: "SB,SB,SB,W\n"
- note removed: "SB,SB,SB,Y\n"
- note removed: "SB,SB,W\n"
- note removed: "SB,SB,Y\n"
- note removed: "SB,Y,BL\n"
- note removed: "SB,Y,R\n"
- note removed: "SB,Y,W\n"
- note removed: "SB,Y,Y,BL\n"
- note removed: "SB,Y,Y,Y\n"
- note removed: "SB,Y,Y\n"
- note removed: "Standard Volvo Penta Plugs\nSB= Black, GR= Grey, W= White\nR= Red, BN= Brown, Y= Yellow\nP= Pink, BL= Blue, GN= Green\nOR= Orange, VO= Violet"
- note removed: "Wire codes. SB,BL,Y,R,W\nCode always starts with SB. \nSecond code marks the connector, \n3rd and 4th code marks the wire.\nAll these wires will probably be in a single conduit."
- note removed: "WiringWithControlBoard"
- moved on the sheet: D3, D6, D9, P1, P8, Q5, R3, R8, R9
